File: plaqueta/plaqueta.kicad_sch (KiCad schematic)
At the start: 4 parts, among them J1 Conn_01x08_Female, J2 Conn_01x04_Female, J3 POWER, U1 ESP32_DevKit_V1_DOIT

Commit message: updates for eb
Parts:
- added D1: 1N4007, Diode_THT:D_DO-41_SOD81_P10.16mm_Horizontal, symbol Diode:1N4007
- added J4: BORN_RELAY, kicad_user_libraries:tblock_2x1, symbol Connector:Screw_Terminal_01x02
- added K1: FINDER-36.11, Relay_THT:Relay_SPDT_Finder_36.11, symbol Relay:FINDER-36.11
- added Q1: BC337, kicad_user_libraries:krapp-TO-92_HandSolder, symbol Transistor_BJT:BC337
- added R1: 10k, kicad_user_libraries:krapp-res-generic, symbol Device:R
- J2: footprint Connector_PinHeader_2.54mm:PinHeader_1x04_P2.54mm_Vertical -> Connector_PinSocket_2.54mm:PinSocket_1x04_P2.54mm_Vertical
Connections:
- net +5V: now also J3.1 (Pin_1), D1.1 (K), K1.A1
- net GND: now also J3.2 (Pin_2), Q1.3 (E)
- net RST/Reset: now also U1.29 (IO22); no longer U1.26 (IO21)
- net at U1.21 (IO16): no longer J2.3 (Pin_3)
- net at U1.22 (IO17): no longer J2.4 (Pin_4)
- net I2C_SCL: now reaches U1.10 (IO27)
- net I2C_SCL: now also J2.3 (Pin_3)
- net at U1.19 (IO2): now also R1.1
- net I2C_SDA: now reaches U1.9 (IO26)
- net I2C_SDA: now also J2.4 (Pin_4)
- new net: D1.2 (A), K1.A2, Q1.1 (C)
- new net: Q1.2 (B), R1.2
- new net: J4.1 (Pin_1), K1.11
- new net: J4.2 (Pin_2), K1.14

Commit message: actualizado el informe
Other:
- moved on the sheet: D1, J1, J2, J3, J4, K1, Q1, R1, U1
